Commit message: joint for left wheel implemented, need to sort out origin and exactly how it offsets...

File: my_rb1_description/urdf/my_rb1_robot.urdf (robot description, URDF)
Before this commit: robot my_rb1_robot, 2 links, 0 joints
Joints:
- added joint joint_chassis_left_wheel: type continuous, parent link_chassis, child left_wheel, origin xyz=0 0.2 -0.15 rpy=0 0 0, axis 0 1 0, limit effort=10000 velocity=1000

Commit message: added the right wheel and joint through copy and paste with text edit to right wheel... need to adjust size, add base frame, and change link_chasis to base_link

File: my_rb1_description/urdf/my_rb1_robot.urdf (robot description, URDF)
Before this commit: robot my_rb1_robot, 2 links, 1 joints
Links:
- added link right_wheel, mass 1; collision cylinder length=0.025 radius=.025; visual cylinder length=.025 radius=.025
Joints:
- added joint joint_chassis_right_wheel: type continuous, parent link_chassis, child right_wheel, origin xyz=0 -0.2 -0.15 rpy=0 0 0, axis 0 1 0, limit effort=10000 velocity=1000

Commit message: placed one caster wheel, size seems odd but placed alright thus far... still working on the origin and joint reference understanding. Will need to add other caster and laser.

File: my_rb1_description/urdf/my_rb1_robot.urdf (robot description, URDF)
Before this commit: robot my_rb1_robot, 3 links, 2 joints
Links:
- added link base_frame, mass 0; collision cylinder length=0 radius=0; visual cylinder length=0 radius=0
- added link front_caster_wheel, mass 1; collision sphere radius=0.025; collision sphere radius=0.05
- link left_wheel: geometry collision cylinder length=0.04 radius=.025; visual cylinder length=.04 radius=.025
- link right_wheel: geometry collision cylinder length=0.04 radius=.025; visual cylinder length=.04 radius=.025
Joints:
- added joint joint_chassis_base_frame: type fixed, parent link_chassis, child base_frame, origin xyz=0 0 -0.15 rpy=0 0 0, axis 0 0 0, limit effort=10000 velocity=1000
- added joint joint_chassis_front_caster_wheel: type fixed, parent link_chassis, child front_caster_wheel, origin xyz=0.1 0 -0.15 rpy=0 0 0

Commit message: added a new caster and changed the name of link_chassis to base_link

File: my_rb1_description/urdf/my_rb1_robot.urdf (robot description, URDF)
Before this commit: robot my_rb1_robot, 5 links, 4 joints
Links:
- removed link front_caster_wheel
- removed link link_chassis
- added link back_caster, mass 1; collision sphere radius=0.025; collision sphere radius=0.05
- added link base_link, mass 25; collision cylinder length=0.30 radius=0.25; visual cylinder length=0.30 radius=0.25
- added link front_caster, mass 1; collision sphere radius=0.025; collision sphere radius=0.05
Joints:
- removed joint joint_chassis_front_caster_wheel
- added joint joint_chassis_back_caster: type fixed, parent base_link, child back_caster, origin xyz=-0.1 0 -0.15 rpy=0 0 0
- added joint joint_chassis_front_caster: type fixed, parent base_link, child front_caster, origin xyz=0.1 0 -0.15 rpy=0 0 0
- joint joint_chassis_base_frame: parent link_chassis -> base_link
- joint joint_chassis_left_wheel: parent link_chassis -> base_link
- joint joint_chassis_right_wheel: parent link_chassis -> base_link

Commit message: added laser and now working to add moments of inertias... treating them as simple objects rotating around a larger one and a cylinder... not sure if I can have each have their own moment of inertia or should i be summating them??

File: my_rb1_description/urdf/my_rb1_robot.urdf (robot description, URDF)
Before this commit: robot my_rb1_robot, 6 links, 5 joints
Links:
- removed link base_frame
- added link base_footprint, mass 0; collision cylinder length=0 radius=0; visual cylinder length=0 radius=0
- added link front_laser, mass 0.5; collision cylinder length=0.02 radius=0.025; visual cylinder length=0.02 radius=0.025
Joints:
- removed joint joint_chassis_base_frame
- added joint joint_chassis_base_footprint: type fixed, parent base_link, child base_footprint, origin xyz=0 0 -0.15 rpy=0 0 0, axis 0 0 0, limit effort=10000 velocity=1000
- added joint joint_chassis_front_laser: type fixed, parent base_link, child front_laser, origin xyz=0.25 0 0.075 rpy=3.14159 0 0
